Commit message: Structure change, forklift services, image processing, and navigation
Control services sources are now in pioneer_control package
Forklift movements are now ros services
Create Image processing service
Create shop floor guide lines
Create navigation service
Camera position adjustment

File: pioneer_description/urdf/pioneer3dx_mod.xacro (robot description, xacro)
@@ -313,5 +313,5 @@
 	</joint>
   <joint name="camera_joint" type="fixed">
-    <origin xyz="0.18 0 -0.12" rpy="0 1 0"/>
+    <origin xyz="0.18 0 -0.12" rpy="0 1.57 0"/>
     <parent link="top_plate"/>
     <child link="camera_link"/>
@@ -361,5 +361,5 @@
     </visual>
     <inertial>
-      <mass value="1e-5" />
+      <mass value="5e-1" />
       <origin xyz="0 0 0" rpy="0 0 0"/>
       <inertia ixx="1e-6" ixy="0" ixz="0" iyy="1e-6" iyz="0" izz="1e-6" />
@@ -389,5 +389,5 @@
     </visual>
     <inertial>
-      <mass value="1e-2" />
+      <mass value="4e-1" />
       <origin xyz="0 0 0" rpy="0 0 0"/>
       <inertia ixx="1e-6" ixy="0" ixz="0" iyy="1e-6" iyz="0" izz="1e-6" />
@@ -414,5 +414,5 @@
     </visual>
     <inertial>
-      <mass value="1e-5" />
+      <mass value="3e-1" />
       <origin xyz="0 0 0" rpy="0 0 0"/>
       <inertia ixx="1e-6" ixy="0" ixz="0" iyy="1e-6" iyz="0" izz="1e-6" />
@@ -439,5 +439,5 @@
     </visual>
     <inertial>
-      <mass value="1e-5" />
+      <mass value="1e-1" />
       <origin xyz="0 0 0" rpy="0 0 0"/>
       <inertia ixx="1e-6" ixy="0" ixz="0" iyy="1e-6" iyz="0" izz="1e-6" />
@@ -464,5 +464,5 @@
     </visual>
     <inertial>
-      <mass value="1e-5" />
+      <mass value="1e-1" />
       <origin xyz="0 0 0" rpy="0 0 0"/>
       <inertia ixx="1e-6" ixy="0" ixz="0" iyy="1e-6" iyz="0" izz="1e-6" />

File: pioneer_description/urdf/pioneer3dx_multi.xacro (robot description, xacro)
@@ -318,5 +318,5 @@
 	</joint>
   <joint name="camera_joint" type="fixed">
-    <origin xyz="0.18 0 -0.12" rpy="0 1 0"/>
+    <origin xyz="0.21 0 -0.13" rpy="0 1.55 0"/>
     <parent link="top_plate"/>
     <child link="camera_link"/>
@@ -327,5 +327,5 @@
       <origin xyz="0 0 0" rpy="0 0 0"/>
       <geometry>
-	      <box size="0.05 0.07 0.10"/>
+	      <box size="0.05 0.07 0.07"/>
       </geometry>
     </collision>
@@ -333,5 +333,5 @@
       <origin xyz="0 0 0" rpy="0 0 0"/>
       <geometry>
-      	<box size="0.05 0.07 0.10"/>
+      	<box size="0.05 0.07 0.07"/>
       </geometry>
       <material name="CameraGreen"/>
@@ -346,6 +346,5 @@
   <joint name="fork_vertical_base_joint" type="fixed">
     <axis xyz="0 1 0"/>
-    <limit effort="1000.0" lower="-0.5" upper="0.5" velocity="1.0"/>
-    <origin xyz="0.2 0 0.01" rpy="0 0 0"/>
+    <origin xyz="0.245 0 0.124" rpy="0 -0.01 0"/>
     <parent link="top_plate"/>
     <child link="fork_vertical_base"/>
@@ -353,13 +352,13 @@
   <link name="fork_vertical_base">
     <collision>
-       <origin xyz="0.02 0 0.11" rpy="0 0 0"/>
-      <geometry>
-	      <box size="0.018 0.05 0.25"/>
+       <origin xyz="0 0 0" rpy="0 0 0"/>
+      <geometry>
+	      <box size="0.04 0.05 0.25"/>
       </geometry>
    </collision>
     <visual>
-      <origin xyz="0.02 0 0.11" rpy="0 0 0"/>
-      <geometry>
-	      <box size="0.018 0.05 0.25"/>
+      <origin xyz="0 0 0" rpy="0 0 0"/>
+      <geometry>
+	      <box size="0.04 0.05 0.25"/>
       </geometry>
      <material name="CameraGreen"/>
@@ -374,6 +373,6 @@
   <joint name="fork_moving_base_joint" type="prismatic">
     <axis xyz="0 0 1"/>
-    <limit effort="1000.0" lower="-0.15" upper="0.2" velocity="1.0"/>
-    <origin xyz="0 0 0" rpy="0 0 0"/>
+    <limit effort="1000.0" lower="-0.15" upper="0.2" velocity="0.3"/>
+    <origin xyz="0.028 0 -0.02" rpy="0 0 0"/>
     <parent link="fork_vertical_base"/>
     <child link="fork_moving_base"/>
@@ -381,11 +380,11 @@
   <link name="fork_moving_base">
     <collision>
-       <origin xyz="0.03 0 0.08" rpy="0 0 0"/>
-      <geometry>
-	      <box size="0.018 0.03 0.3"/>
+       <origin xyz="0 0 0" rpy="0 0 0"/>
+      <geometry>
+        <box size="0.018 0.03 0.3"/>
       </geometry>
    </collision>
     <visual>
-      <origin xyz="0.03 0 0.08" rpy="0 0 0"/>
+      <origin xyz="0 0 0" rpy="0 0 0"/>
       <geometry>
 	      <box size="0.018 0.03 0.3"/>
@@ -403,8 +402,9 @@
     <parent link="fork_moving_base"/>
     <child link="fork_horizontal_base"/>
+     <origin xyz="0.002 0 -0.175" rpy="0 0 0"/>
   </joint>
   <link name="fork_horizontal_base">
     <collision>
-       <origin xyz="0.036 0 -0.08" rpy="0 0 0"/>
+      <origin xyz="0 0 0" rpy="0 0 0"/>
       <geometry>
 	      <box size="0.018 0.2 0.05"/>
@@ -412,5 +412,5 @@
    </collision>
     <visual>
-      <origin xyz="0.036 0 -0.08" rpy="0 0 0"/>
+      <origin xyz="0 0 0" rpy="0 0 0"/>
       <geometry>
 	      <box size="0.018 0.2 0.05"/>
@@ -428,8 +428,9 @@
     <parent link="fork_horizontal_base"/>
     <child link="left_fork"/>
+    <origin xyz="0.095 0.075 -0.023" rpy="0 -0.035 0"/>
   </joint>
   <link name="left_fork">
   <collision>
-       <origin xyz="0.13 0.075 -0.096" rpy="0 -0.05 0"/>
+       <origin xyz="0 0 0" rpy="0 0 0"/>
       <geometry>
 	      <box size="0.20 0.05 0.01"/>
@@ -437,5 +438,5 @@
    </collision>
     <visual>
-      <origin xyz="0.13 0.075 -0.096" rpy="0 -0.05 0"/>
+      <origin xyz="0 0 0" rpy="0 0 0"/>
       <geometry>
 	      <box size="0.20 0.05 0.01"/>
@@ -453,8 +454,9 @@
     <parent link="fork_horizontal_base"/>
     <child link="right_fork"/>
+    <origin xyz="0.095 -0.075 -0.023" rpy="0 -0.035 0"/>
   </joint>
   <link name="right_fork">
     <collision>
-      <origin xyz="0.13 -0.075 -0.096" rpy="0 -0.05 0"/>
+      <origin xyz="0 0 0" rpy="0 0 0"/>
       <geometry>
 	      <box size="0.20 0.05 0.01"/>
@@ -462,7 +464,7 @@
    </collision>
     <visual>
-      <origin xyz="0.13 -0.075 -0.096" rpy="0 -0.05 0"/>
-      <geometry>
-	      <box size="0.20 0.05 0.01"/>
+      <origin xyz="0 0 0" rpy="0 0 0"/>
+      <geometry>
+	      <box size="0.2 0.05 0.01"/>
       </geometry>
       <material name="CameraGreen"/>
@@ -475,8 +477,9 @@
   </link>
 <!-- Counterweight -->
+<!-- inside the chassis over the swivel for stability-->
   <joint name="counterweight_joint" type="fixed">
-    <origin xyz="-0.18 0 -0.025" rpy="0 0 0"/>
     <parent link="chassis"/>
     <child link="counterweight_base"/>
+    <origin xyz="-0.05 0 -0.025" rpy="0 0 0"/>
   </joint>
   <link name="counterweight_base">
@@ -494,5 +497,5 @@
     </visual>
     <inertial>
-      <mass value="5" />
+      <mass value="4" />
       <origin xyz="0 0 0" rpy="0 0 0"/>
       <inertia ixx="0" ixy="0" ixz="0" iyy="0" iyz="0" izz="0" />

File: stage_assets/assets/product.xacro (robot description, xacro)
@@ -9,11 +9,11 @@
 <xacro:property name="base_length" value="0.007"/>
 <xacro:property name="base_radius" value="0.08"/>
-<xacro:property name="base_mass" value="0.2"/>
+<xacro:property name="base_mass" value="0.05"/>
 <xacro:property name="pick_up_length" value="0.04"/>
 <xacro:property name="pick_up_radius" value="0.035"/>
-<xacro:property name="pick_up_mass" value="0.05"/>
+<xacro:property name="pick_up_mass" value="0.01"/>
 <xacro:property name="product_length" value="0.35"/>
 <xacro:property name="product_radius" value="0.09"/>
-<xacro:property name="product_mass" value="0.2"/>
+<xacro:property name="product_mass" value="0.05"/>
 <link name="base">
   <visual>
